Commit message: xacro_caster

File: urdf/my_robot.urdf.xacro (robot description, xacro)
@@ -6,4 +6,8 @@
     <xacro:property name="length" value="0.02"/>
     <xacro:property name="wheel_mass" value="2.5" /> <!-- in kg-->
+    <xacro:property name="base_x_origin_to_caster_front_origin" value="0.115"/>
+    <xacro:property name="base_z_origin_to_caster_front" value="0.007"/>
+    <xacro:property name="base_x_origin_to_caster_back_origin" value="-0.135"/>
+    <xacro:property name="base_z_origin_to_caster_back" value="0.009"/>
     <xacro:macro name="cylinder_inertia" params="m r h">
         <inertial>
@@ -13,4 +17,13 @@
               iyy="${m*(3*r*r+h*h)/12}" iyz = "0"
               izz="${m*r*r/2}" />
+        </inertial>
+    </xacro:macro>
+    <xacro:macreo name="caster_inertia" params="m r">
+        <inertial>
+            <mass value="${m}"/>
+            <origin xyz="0 0 0"/>
+            <inertia ixx="${(2*m*r*r)/5}" ixy="0" ixz="0"
+                iyy="${(2*m*r*r)/5}" iyz="0"
+                izz="${(2*m*r*r)/5}" />
         </inertial>
     </xacro:macro>
@@ -33,5 +46,5 @@
     </xacro:macro>
     <xacro:macro name="caster_wheel" params= "fb parent translateX translateY">
-        <link name="${fb}_wheel">
+        <link name="caster_${fb}_wheel">
             <visual>
                 <origin xyz="0 0 0" rpy="0 0 0"/>
@@ -40,5 +53,17 @@
                 </geometry>
             </visual>
+            <collision>
+                <origin xyz="0 0 0" rpy="0 0 0"/>
+                <geometry>
+                    <sphere radius="${radius_caster}"/>
+                </geometry>
+            </collision>
+            <caster_inertia m="${wheel_mass}" r="${radius_caster}"/>
         </link>
+        <joint name="caster_${fb}_joint" type="continuous">
+            <parent link="${parent}"/>
+            <child link="caster_${fb}_wheel"/>
+            <origin xyz="${translateX * base_x_origin_to_caster_${fb}_origin} 0 ${base_z_origin_to_caster_${fb}}" rpy="-1.57 0 0"/>
+        </joint>
     </xacro:macro>
 </robot>

Commit message: joint_gazebo_wheel_cyl

File: urdf/my_robot.urdf.xacro (robot description, xacro)
@@ -6,4 +6,5 @@
     <xacro:property name="length" value="0.02"/>
     <xacro:property name="wheel_mass" value="2.5" /> <!-- in kg-->
+    <xacro:property name="base_y_origin_to_wheel_origin" value="0.15"/>
     <xacro:macro name="cylinder_inertia" params="m r h">
         <inertial>
@@ -31,4 +32,21 @@
       <cylinder_inertia m="${wheel_mass}" r="${radius_wheel}" h="${length}" />
     </link>
+    <gazebo reference="${lr}_wheel">
+      <mu1 value="1.0"/>
+      <mu2 value="1.0"/>
+      <kp value="10000000.0"/>
+      <kd value="1.0"/>
+      <fdir1 value="1.0"/>Gra
+      <material>Gazebo/grey</material>
+      <turnGravityOff>false</turnGravityOff>
+    </gazebo>
+    <joint name="${lr}_wheel_joint" type="continuous">
+      <parent link="${parent}"/>
+      <child link="${lr}_wheel"/>
+      <origin xyz="0 ${translateY*base_y_to_origin_to_wheel_origin} 0}" rpy="0 0 0"/>
+      <axis xyz="0 1 0" rpy="0 0"/>
+      <limit effort="100" velocity="100"/>
+      <joint_properties damping="0.0" friction="0.0"/>
+    </joint>
     </xacro:macro>
     <xacro:macro name="caster_wheel" params= "fb parent translateX translateY">

Commit message: xacro-correggere caster macro fb

File: urdf/my_robot.urdf.xacro (robot description, xacro)
@@ -1,4 +1,4 @@
 <?xml version="1.0"?>
-<robot name="my_robot">
+<robot name="my_robot" xmlns:xacro="http://www.ros.org/wiki/xacro">
     <xacro:property name="pi" value="3.1415" />
     <xacro:property name="radius_wheel" value="0.04"/>
@@ -20,5 +20,5 @@
         </inertial>
     </xacro:macro>
-    <xacro:macreo name="caster_inertia" params="m r">
+    <xacro:macro name="caster_inertia" params="m r">
         <inertial>
             <mass value="${m}"/>
@@ -29,5 +29,5 @@
         </inertial>
     </xacro:macro>
-    <xacro:macro name="cylinder_wheel" params="fb lr parent translateX translateY flipY"> <!--fb : front, back ; lr: left, right -->
+    <xacro:macro name="cylinder_wheel" params="lr parent translateX translateY flipY"> <!--fb : front, back ; lr: left, right -->
          <link name="${lr}_wheel">
       <visual>
@@ -50,6 +50,5 @@
       <kp value="10000000.0"/>
       <kd value="1.0"/>
-      <fdir1 value="1.0"/>Gra
-      <material>Gazebo/grey</material>
+      <fdir1 value="1.0"/>
       <turnGravityOff>false</turnGravityOff>
     </gazebo>
@@ -57,14 +56,14 @@
       <parent link="${parent}"/>
       <child link="${lr}_wheel"/>
-      <origin xyz="0 ${translateY*base_y_to_origin_to_wheel_origin} 0}" rpy="0 0 0"/>
-      <axis xyz="0 1 0" rpy="0 0"/>
+      <origin xyz="0 ${translateY*base_y_origin_to_wheel_origin} 0" rpy="0 0 0"/>
+      <axis xyz="0 1 0" rpy="0 0 0"/>
       <limit effort="100" velocity="100"/>
       <joint_properties damping="0.0" friction="0.0"/>
     </joint>
     </xacro:macro>
-    <xacro:macro name="caster_wheel" params= "fb parent translateX translateY">
+    <xacro:macro name="caster_wheel" params= "fb parent translateX">   <!--translateX=0 per front translateX=1 per back-->
         <link name="caster_${fb}_wheel">
             <visual>
-                <origin xyz="0 0 0" rpy="0 0 0"/>
+                <origin xyz="${translateX*0.02}  0.02 0" rpy="1.57 0 0"/>
                 <geometry>
                     <sphere radius="${radius_caster}"/>
@@ -72,5 +71,5 @@
             </visual>
             <collision>
-                <origin xyz="0 0 0" rpy="0 0 0"/>
+                <origin xyz="${translateX*0.02}  0.02 0" rpy="1.57 0 0"/>
                 <geometry>
                     <sphere radius="${radius_caster}"/>
@@ -82,6 +81,35 @@
             <parent link="${parent}"/>
             <child link="caster_${fb}_wheel"/>
-            <origin xyz="${translateX * base_x_origin_to_caster_${fb}_origin} 0 ${base_z_origin_to_caster_${fb}}" rpy="-1.57 0 0"/>
+            <origin xyz="${base_x_origin_to_caster_${fb}_origin} 0 ${base_z_origin_to_caster_${fb}}" rpy="-1.57 0 0"/>
         </joint>
+        <gazebo reference="caster_${fb}_wheel">
+            <mu1 value="1.0"/>
+            <mu2 value="1.0"/>
+            <kp  value="10000000.0" />
+            <kd  value="1.0" />
+            <fdir1 value="1 0 0"/>
+            <turnGravityOff>false</turnGravityOff>
+        </gazebo>
     </xacro:macro>
+    <link name="base_link">
+        <visual>
+        <geometry>
+            <cylinder length="0.15" radius="0.02"/>
+        </geometry>
+        <origin rpy= "0 0 0" xyz= "0 0 0" />
+        </visual>
+        <cylinder_inertia m="5" r="0.02" h="0.15" />
+    </link>
+    <gazebo reference="base_link">
+        <mu1 value="1.0"/>
+        <mu2 value="1.0"/>
+        <kp  value="10000000.0" />
+        <kd  value="1.0" />
+        <fdir1 value="1 0 0"/>
+        <turnGravityOff>false</turnGravityOff>
+    </gazebo>
+    <cylinder_wheel  lr="left" parent="base_link" translateX="0" translateY="0.5" flipY="1" />
+    <cylinder_wheel  lr="right" parent="base_link" translateX="0" translateY="-0.5" flipY="1" />
+    <caster_wheel fb="front" parent="base_link" translateX="0" />
+    <caster_wheel fb="front" parent="base_link" translateX="1" />
 </robot>

Commit message: gazebo.launch- dimensioni non corrette

File: urdf/my_robot.urdf.xacro (robot description, xacro)
@@ -6,8 +6,8 @@
     <xacro:property name="length" value="0.02"/>
     <xacro:property name="wheel_mass" value="2.5" /> <!-- in kg-->
-    <xacro:property name="base_x_origin_to_caster_front_origin" value="0.115"/>
+<!--     <xacro:property name="base_x_origin_to_caster_front_origin" value="0.115"/>
     <xacro:property name="base_z_origin_to_caster_front" value="0.007"/>
     <xacro:property name="base_x_origin_to_caster_back_origin" value="-0.135"/>
-    <xacro:property name="base_z_origin_to_caster_back" value="0.009"/>
+    <xacro:property name="base_z_origin_to_caster_back" value="0.009"/> -->
     <xacro:property name="base_y_origin_to_wheel_origin" value="0.15"/>
     <xacro:macro name="cylinder_inertia" params="m r h">
@@ -43,5 +43,5 @@
         </geometry>
       </collision>
-      <cylinder_inertia m="${wheel_mass}" r="${radius_wheel}" h="${length}" />
+      <xacro:cylinder_inertia m="${wheel_mass}" r="${radius_wheel}" h="${length}" />
     </link>
     <gazebo reference="${lr}_wheel">
@@ -62,5 +62,5 @@
     </joint>
     </xacro:macro>
-    <xacro:macro name="caster_wheel" params= "fb parent translateX">   <!--translateX=0 per front translateX=1 per back-->
+    <xacro:macro name="caster_wheel" params= "fb parent translateX base_x_origin_to_caster_origin base_z_origin_to_caster_origin">   <!--translateX=0 per front translateX=1 per back-->
         <link name="caster_${fb}_wheel">
             <visual>
@@ -76,10 +76,10 @@
                 </geometry>
             </collision>
-            <caster_inertia m="${wheel_mass}" r="${radius_caster}"/>
+            <xacro:caster_inertia m="${wheel_mass}" r="${radius_caster}"/>
         </link>
         <joint name="caster_${fb}_joint" type="continuous">
             <parent link="${parent}"/>
             <child link="caster_${fb}_wheel"/>
-            <origin xyz="${base_x_origin_to_caster_${fb}_origin} 0 ${base_z_origin_to_caster_${fb}}" rpy="-1.57 0 0"/>
+            <origin xyz="${base_x_origin_to_caster_origin} 0 ${base_z_origin_to_caster_origin}" rpy="-1.57 0 0"/>
         </joint>
         <gazebo reference="caster_${fb}_wheel">
@@ -99,5 +99,5 @@
         <origin rpy= "0 0 0" xyz= "0 0 0" />
         </visual>
-        <cylinder_inertia m="5" r="0.02" h="0.15" />
+        <xacro:cylinder_inertia m="5" r="0.02" h="0.15" />
     </link>
     <gazebo reference="base_link">
@@ -109,7 +109,7 @@
         <turnGravityOff>false</turnGravityOff>
     </gazebo>
-    <cylinder_wheel  lr="left" parent="base_link" translateX="0" translateY="0.5" flipY="1" />
-    <cylinder_wheel  lr="right" parent="base_link" translateX="0" translateY="-0.5" flipY="1" />
-    <caster_wheel fb="front" parent="base_link" translateX="0" />
-    <caster_wheel fb="front" parent="base_link" translateX="1" />
+    <xacro:cylinder_wheel  lr="left" parent="base_link" translateX="0" translateY="0.5" flipY="1" />
+    <xacro:cylinder_wheel  lr="right" parent="base_link" translateX="0" translateY="-0.5" flipY="1" />
+    <xacro:caster_wheel fb="front" parent="base_link" translateX="0" base_x_origin_to_caster_origin="0.115" base_z_origin_to_caster_origin="0.007" />
+    <xacro:caster_wheel fb="back" parent="base_link" translateX="1" base_x_origin_to_caster_origin="0.135" base_z_origin_to_caster_origin="0.009" />
 </robot>

Commit message: spawn_robot_corretto

File: urdf/my_robot.urdf.xacro (robot description, xacro)
@@ -78,5 +78,5 @@
             <xacro:caster_inertia m="${wheel_mass}" r="${radius_caster}"/>
         </link>
-        <joint name="caster_${fb}_joint" type="continuous">
+        <joint name="caster_${fb}_joint" type="fixed">
             <parent link="${parent}"/>
             <child link="caster_${fb}_wheel"/>
@@ -95,9 +95,9 @@
         <visual>
         <geometry>
-            <cylinder length="0.15" radius="0.02"/>
+            <cylinder length="0.02" radius="0.15"/>
         </geometry>
         <origin rpy= "0 0 0" xyz= "0 0 0" />
         </visual>
-        <xacro:cylinder_inertia m="5" r="0.02" h="0.15" />
+        <xacro:cylinder_inertia m="5" r="0.15" h="0.02" />
     </link>
     <gazebo reference="base_link">
@@ -112,4 +112,4 @@
     <xacro:cylinder_wheel  lr="right" parent="base_link" translateX="0" translateY="-0.5" flipY="1" />
     <xacro:caster_wheel fb="front" parent="base_link" translateX="0" base_x_origin_to_caster_origin="0.115" base_z_origin_to_caster_origin="0.007" />
-    <xacro:caster_wheel fb="back" parent="base_link" translateX="1" base_x_origin_to_caster_origin="0.135" base_z_origin_to_caster_origin="0.009" />
+    <xacro:caster_wheel fb="back" parent="base_link" translateX="1" base_x_origin_to_caster_origin="-0.135" base_z_origin_to_caster_origin="0.009" />
 </robot>

Commit message: creazione_yaml

File: urdf/my_robot.urdf.xacro (robot description, xacro)
@@ -31,34 +31,43 @@
     <xacro:macro name="cylinder_wheel" params="lr parent translateX translateY flipY"> <!--fb : front, back ; lr: left, right -->
          <link name="${lr}_wheel">
-      <visual>
-        <origin xyz="0 0 0" rpy="${flipY*pi/2} 0  0 " />
-        <geometry>
-          <cylinder length="${length}" radius="${radius_wheel}" />
-        </geometry>
-      </visual>
-      <collision>
-        <origin xyz="0 0 0" rpy="${flipY*pi/2} 0 0 " />
-        <geometry>
-          <cylinder length="${length}" radius="${radius_wheel}" />
-        </geometry>
-      </collision>
-      <xacro:cylinder_inertia m="${wheel_mass}" r="${radius_wheel}" h="${length}" />
-    </link>
-    <gazebo reference="${lr}_wheel">
-      <mu1 value="1.0"/>
-      <mu2 value="1.0"/>
-      <kp value="10000000.0"/>
-      <kd value="1.0"/>
-      <fdir1 value="1.0"/>
-      <turnGravityOff>false</turnGravityOff>
-    </gazebo>
-    <joint name="${lr}_wheel_joint" type="continuous">
-      <parent link="${parent}"/>
-      <child link="${lr}_wheel"/>
-      <origin xyz="0 ${translateY*base_y_origin_to_wheel_origin} 0" rpy="0 0 0"/>
-      <axis xyz="0 1 0" rpy="0 0 0"/>
-      <limit effort="100" velocity="100"/>
-      <joint_properties damping="0.0" friction="0.0"/>
-    </joint>
+            <visual>
+                <origin xyz="0 0 0" rpy="${flipY*pi/2} 0  0 " />
+                <geometry>
+                <cylinder length="${length}" radius="${radius_wheel}" />
+                </geometry>
+            </visual>
+            <collision>
+                <origin xyz="0 0 0" rpy="${flipY*pi/2} 0 0 " />
+                <geometry>
+                <cylinder length="${length}" radius="${radius_wheel}" />
+                </geometry>
+            </collision>
+            <xacro:cylinder_inertia m="${wheel_mass}" r="${radius_wheel}" h="${length}" />
+        </link>
+        <gazebo reference="${lr}_wheel">
+            <mu1 value="1.0"/>
+            <mu2 value="1.0"/>
+            <kp value="10000000.0"/>
+            <kd value="1.0"/>
+            <fdir1 value="1.0"/>
+            <turnGravityOff>false</turnGravityOff>
+        </gazebo>
+        <joint name="${lr}_wheel_joint" type="continuous">
+            <parent link="${parent}"/>
+            <child link="${lr}_wheel"/>
+            <origin xyz="0 ${translateY*base_y_origin_to_wheel_origin} 0" rpy="0 0 0"/>
+            <axis xyz="0 1 0" rpy="0 0 0"/>
+            <limit effort="100" velocity="100"/>
+            <joint_properties damping="0.0" friction="0.0"/>
+        </joint>
+        <transmission name="${lr}_wheel_joint_trans">
+            <type>transmission_interface/simpleTransmission</type>
+            <joint name="${lr}_wheel_joint">
+                <hardwareInterface>hardware_interface/VelocityJointInterface</hardwareInterface>
+            </joint>
+            <actuator name="${lr}_wheel_joint_motor">
+                <mechanicalReduction>1</mechanicalReduction>
+            </actuator>
+        </transmission>
     </xacro:macro>
     <xacro:macro name="caster_wheel" params= "fb parent translateX base_x_origin_to_caster_origin base_z_origin_to_caster_origin">   <!--translateX=0 per front translateX=1 per back-->
@@ -113,3 +122,8 @@
     <xacro:caster_wheel fb="front" parent="base_link" translateX="0" base_x_origin_to_caster_origin="0.115" base_z_origin_to_caster_origin="0.007" />
     <xacro:caster_wheel fb="back" parent="base_link" translateX="1" base_x_origin_to_caster_origin="-0.135" base_z_origin_to_caster_origin="0.009" />
+    <gazebo>
+        <plugin name="gazebo_ros_control" filename="libgazebo_ros_control.so">
+            <robotNamespace>my_robot</robotNamespace>
+        </plugin>
+    </gazebo>
 </robot>
